File: pcb/pcb.kicad_pcb (KiCad board)
At the start: 2 copper layers, 74 x 12.7 mm, 20 parts, among them J0 Qwiic, J1 Qwiic, J2 Conn_01x12, U1 AT42QT2120-SU

Commit message: Second stab at a PCB
Parts:
- removed R0, R10, R11, R4, R5, R6, R7, R8, R9: 4.7k, Resistor_SMD:R_0805_2012Metric_Pad1.20x1.40mm_HandSolder
- removed the R1 at (160.0, 108.2)
- removed the R2 at (157.5, 108.2)
- removed the R3 at (154.9, 108.2)
- added J3: Conn_01x12, Connector_Wire:SolderWire-0.1sqmm_1x04_P3.6mm_D0.4mm_OD1mm, F.Cu at (143.0, 109.1)
- added J4: Conn_01x12, Connector_Wire:SolderWire-0.1sqmm_1x04_P3.6mm_D0.4mm_OD1mm, F.Cu at (143.0, 112.8)
- added RN1: 4.7k, Package_SO:SSOP-24_3.9x8.7mm_P0.635mm, F.Cu at (148.8, 109.0)
- J2: footprint Connector_PinHeader_2.54mm:PinHeader_1x12_P2.54mm_Vertical -> Connector_Wire:SolderWire-0.1sqmm_1x04_P3.6mm_D0.4mm_OD1mm
- moved J2 19.6 mm to (143.0, 105.4), turned to 180 degrees
- moved J0 14.5 mm to (176.5, 108.7)
- moved R1 13.0 mm to (169.4, 109.7)
- moved R3 13.0 mm to (169.4, 107.7)
- moved C0 13.0 mm to (169.4, 111.8)
- moved R2 13.0 mm to (169.4, 105.7)
- moved U1 12.8 mm to (159.8, 109.0)
- moved J1 0.58 mm to (126.5, 108.7)
- renumbered R12 to R1, R13 to R2, R14 to R3
Routing:
- net Net-(U1-Pad18): track 39.0 -> 5.99 mm, vias 2 -> 0
- net Net-(U1-Pad19): track 34.9 -> 4.46 mm, vias 2 -> 0
- net Net-(U1-Pad20): track 30.6 -> 3.09 mm, vias 2 -> 0
- net Net-(U1-Pad1): track 26.8 -> 3.09 mm
- net Net-(U1-Pad2): track 25.7 -> 4.46 mm
- net Net-(U1-Pad3): track 24.4 -> 5.99 mm
- net Net-(RN1-Pad12): track 0.00 -> 15.7 mm
- net Net-(U1-Pad4): track 23.1 -> 7.52 mm
- net Net-(RN1-Pad8): track 0.00 -> 15.4 mm
- net +5V: track 74.1 -> 59.8 mm, vias 0 -> 2
- net Net-(J0-Pad4): track 75.8 -> 62.1 mm
- net Net-(U1-Pad5): track 21.8 -> 9.06 mm
- net Net-(RN1-Pad11): track 0.00 -> 12.6 mm
- net Net-(RN1-Pad4): track 2.84 -> 14.9 mm
- net Net-(RN1-Pad7): track 0.00 -> 11.7 mm
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Other:
- board size 74 x 12.7 mm -> 59 x 12.7 mm
