File: pcb/pcb.kicad_sch (KiCad schematic)
At the start: 20 parts, among them J0 Qwiic, J1 Qwiic, J2 Conn_01x12, U1 AT42QT2120-SU

Commit message: Second stab at a PCB
Parts:
- removed J2: Conn_01x12, Connector_PinHeader_2.54mm:PinHeader_1x12_P2.54mm_Vertical, symbol Connector_Generic:Conn_01x12
- removed R0, R1, R10, R11, R2, R3, R4, R5, R6, R7, R8, R9: 4.7k, Resistor_SMD:R_0805_2012Metric_Pad1.20x1.40mm_HandSolder, symbol Device:R_US
- added J2: Conn_01x12, symbol Connector_Generic:Conn_01x04
- added J3, J4: Conn_01x12, Connector_Wire:SolderWire-0.1sqmm_1x04_P3.6mm_D0.4mm_OD1mm, symbol Connector_Generic:Conn_01x04
- added RN1: (no value), Package_SO:SSOP-24_3.9x8.7mm_P0.635mm, symbol Device:R_Pack11
- renumbered R12 to R1, R13 to R2, R14 to R3
Connections:
- net at U1.4 (KEY5/GPO3): now also RN1.19 (R6.2)
- net at U1.9 (KEY0): now also RN1.24 (R1.2)
- net at U1.7 (KEY2/GP00): now also RN1.22 (R3.2)
- net at U1.6 (KEY3/GPO1): now also RN1.21 (R4.2)
- net at U1.2 (KEY7/GPO5): now also RN1.17 (R8.2)
- net at U1.19 (KEY10/GPO8): now also RN1.14 (R11.2)
- net at U1.5 (KEY4/GPO2): now also RN1.20 (R5.2)
- net at U1.8 (KEY1): now also RN1.23 (R2.2)
- net at U1.20 (KEY9/GPO7): now also RN1.15 (R10.2)
- net at U1.1 (KEY8/GPO6): now also RN1.16 (R9.2)
- net at U1.18 (KEY/11/GPO9): now also RN1.13 (R12.2)
- net at U1.3 (KEY6/GPO4): now also RN1.18 (R7.2)
- new net: J2.1 (Pin_1), RN1.1 (R1.1)
- new net: J4.2 (Pin_2), RN1.10 (R10.1)
- new net: J4.3 (Pin_3), RN1.11 (R11.1)
- new net: J4.4 (Pin_4), RN1.12 (R12.1)
- new net: J2.2 (Pin_2), RN1.2 (R2.1)
- new net: J2.3 (Pin_3), RN1.3 (R3.1)
- new net: J2.4 (Pin_4), RN1.4 (R4.1)
- new net: J3.1 (Pin_1), RN1.5 (R5.1)
- new net: J3.2 (Pin_2), RN1.6 (R6.1)
- new net: J3.3 (Pin_3), RN1.7 (R7.1)
- new net: J3.4 (Pin_4), RN1.8 (R8.1)
- new net: J4.1 (Pin_1), RN1.9 (R9.1)
